File: IOB-Signal.sch (EAGLE design)
At the start: 25 parts, among them CON1 RJ45, IC1 74HS139A, Q0 MOSFET-P, Q1 MOSFET-P, Q2 MOSFET-P, Q3 MOSFET-P

Commit message: new IOB format
Parts:
- removed FID2: FIDUCIAL, SPCoast:FIDUCIAL
- removed IOB: IO4-IOBBARE, SPCoast:IO4-IOBBARE
- removed LED0, LED1, LED2, LED3: Y, SPCoast:LED0603-LED
- removed Q0, Q1, Q2, Q3: MOSFET-P, SPCoast:MOSFET-P
- removed R0, R1, R2, R3: 2K2, SPCoast:R0805-RES
- added U$1: CONNECTOR-IO4-IOBBARE, SPCoast:CONNECTOR-IO4-IOBBARE
Connections:
- removed net N$11: Q0.D, R0.2
- removed net N$2: LED0.A, R0.1
- removed net N$3: LED1.A, R1.1
- removed net N$30: Q1.D, R1.2
- removed net N$31: Q2.D, R2.2
- removed net N$32: Q3.D, R3.2
- removed net N$4: LED2.A, R2.1
- removed net N$5: LED3.A, R3.1
- net GND: now also U$1.GND; no longer IOB.GND, LED0.C, LED1.C, LED2.C, LED3.C
- net P1: now also U$1.P1; no longer IOB.P1, Q0.G
- net P2: now also U$1.P2; no longer IOB.P2, Q1.G
- net P3: now also U$1.P3; no longer IOB.P3, Q2.G
- net P4: now also U$1.P4; no longer IOB.P4, Q3.G
- net VCC: now also U$1.5V; no longer IOB.5V, Q0.S, Q1.S, Q2.S, Q3.S
- net VCCIO: now also U$1.VIN; no longer IOB.VIN
Other:
- note added: "2.0"
- note added: "A"
- note removed: "1.0"
- note removed: "B"
